File: schematic/insver/insver.sch (KiCad schematic (older format))
At the start: 5 parts, among them U1 74AC191, U2 74AC191, U3 74AC191, U4 74AC191

Commit message: 。。。
Parts:
- added U5: 74AC00, symbol 74xx:74AC00
- added U6: 74AC08, symbol 74xx:74AC08
- gave numbers to parts that had none: 1
Connections:
- net GND: now also U1.~ (~U), U2.~ (~U), U3.~ (~U), U4.~ (~U)
- net ~WE: now reaches J1.~ (~CS2)
- net ~WE: now also U6.~
- new net: U1.~ (~U), U2.~ (~U), U3.~ (~U), U4.~ (~U), U5.~
- new net: U1.~ (~U), U2.~ (~U), U3.~ (~U), U4.~ (~U), U6.~
- new net: U1.~ (~U), U5.~, U5.~, U6.~
- new net: U2.~ (~U), U5.~
- new net: U2.~ (~U), U5.~, U6.~
- new net: U3.~ (~U), U5.~ (x2)
- new net: U4.~ (~U), U5.~
- new net: U5.~, U6.~
- new net A16: J1.~ (~CS2)
- new net A17: J1.~ (~CS2)
- new net A18: J1.~ (~CS2)
- new net A19: J1.~ (~CS2)
- new net A20: J1.~ (~CS2)
- new net A21: J1.~ (~CS2)
- new net A22: J1.~ (~CS2)
- new net A23: J1.~ (~CS2)
- new net ~CE: J1.~ (~CS2), U5.~
- new net ~RE: J1.~ (~CS2), U6.~
- no-connect marks 0 -> 8
Other:
- note added: "1"
- moved on the sheet: J1, U1, U2, U3, U4

Commit message: 。。。
Parts:
- added C1: 10uF, symbol Device:CP1_Small
- renumbered J1 to JP1
Connections:
- net A00: now also U1.~ (~U)
- net A01: now also U1.~ (~U)
- net A02: now also U1.~ (~U)
- net A03: now also U1.~ (~U)
- net A04: now also U2.~ (~U)
- net A05: now also U2.~ (~U)
- net A06: now also U2.~ (~U)
- net A07: now also U2.~ (~U)
- net A08: now also U3.~ (~U)
- net A09: now also U3.~ (~U)
- net A10: now also U3.~ (~U)
- net A11: now also U3.~ (~U)
- net A12: now also U4.~ (~U)
- net A13: now also U4.~ (~U)
- net A14: now also U4.~ (~U)
- net A15: now also U4.~ (~U)
- net D00: now also U1.~ (~U)
- net D01: now also U1.~ (~U)
- net D02: now also U1.~ (~U)
- net D03: now also U1.~ (~U)
- net D04: now also U2.~ (~U)
- net D05: now also U2.~ (~U)
- net D06: now also U2.~ (~U)
- net D07: now also U2.~ (~U)
- net D08: now also U3.~ (~U)
- net D09: now also U3.~ (~U)
- net D10: now also U3.~ (~U)
- net D11: now also U3.~ (~U)
- net D12: now also U4.~ (~U)
- net D13: now also U4.~ (~U)
- net D14: now also U4.~ (~U)
- net D15: now also U4.~ (~U)
- net GND: now also C1.2
- net VCC: now also C1.1
- net at U5.~: now also U6.~; no longer U3.~ (~U)
- new net: U1.~ (~U), U2.~ (~U), U3.~ (~U), U4.~ (~U), U5.~
- new net: U1.~ (~U), U2.~ (~U), U3.~ (~U), U4.~ (~U), U6.~
- new net: U1.~ (~U), U5.~, U5.~, U6.~
- new net: U2.~ (~U), U5.~, U6.~
- new net: U3.~ (~U), U5.~
- new net: U4.~ (~U), U5.~
- no-connect marks 8 -> 7
Other:
- note added: "12/19/2020\n"
- note added: "A"
- note added: "GBA CARTRIDGE BUS DE-MULTIPLEXER"
- note added: "GBA cartridge bus de-multiplexing and handling \nsequencial bus accessing, using 74191 as counter.\n"
- note removed: "1"
- moved on the sheet: JP1, U1, U2, U3, U4, U5A, U5B, U5C, U5D, U6A, U6B
