File: schematic/insver/insver.sch (KiCad schematic (older format))
At the start: 8 parts, among them U1 74AC191, U2 74AC191, U3 74AC191, U4 74AC191, U5 74AC00, U6 74AC08

Commit message: pin
Connections:
- net ~RE is gone; now on net ~WR: JP1.~ (~CS2), U6.~
- net ~WE is gone; now on net ~WR: JP1.~ (~CS2), U6.~
- net ~WR: now reaches JP1.~ (~CS2)
- net at U5.~: now also U6.~; no longer U3.~ (~U)
- net ~CE renamed ~CS1
- new net: U1.~ (~U), U2.~ (~U), U3.~ (~U), U4.~ (~U), U5.~
- new net: U1.~ (~U), U2.~ (~U), U3.~ (~U), U4.~ (~U), U6.~
- new net: U1.~ (~U), U5.~, U5.~, U6.~
- new net: U2.~ (~U), U5.~, U6.~
- new net: U3.~ (~U), U5.~
- new net: U4.~ (~U), U5.~
- new net ~RD: JP1.~ (~CS2), U6.~
Changed lines of the file:
@@
 A15
 Text GLabel 3350 1800 2    50   Output ~ 0
-~WE
+~WR
 Wire Wire Line
 	2000 1550 2000 1600
-Text GLabel 2700 1600 1    50   Output ~ 0
-~CE
 Text GLabel 3050 1600 1    50   Output ~ 0
-~RE
+~RD
 Wire Wire Line
 	3750 4350 3700 4350
@@
 	3050 1600 3050 1900
 Wire Wire Line
-	2700 1600 2700 2000
-Wire Wire Line
 	2700 4750 3600 4750
 Connection ~ 3600 4750
@@
 Wire Wire Line
 	2700 2000 2700 2900
-Connection ~ 2700 2000
 Connection ~ 2700 2900
 Wire Wire Line
@@
 Text Notes 7150 6850 0    79   ~ 0
 GBA cartridge bus de-multiplexing and handling \nsequencial bus accessing, using 74191 as counter.\n
-Wire Bus Line
-	2300 3800 2300 5250
+Connection ~ 2700 2000
 Wire Bus Line
 	2300 5250 9350 5250
@@
 	2500 2200 10050 2200
 Wire Bus Line
-	2500 2200 2500 3900
-Wire Bus Line
 	10050 2200 10050 3800
 Wire Bus Line
 	9350 2750 9350 5250
+Wire Bus Line
+	2300 3800 2300 5250
+Wire Bus Line
+	2500 2200 2500 3900
+Wire Wire Line
+	2700 1600 2700 2000
+Text GLabel 2700 1600 1    50   Output ~ 0
+~CS1
 $EndSCHEMATC

Commit message: 我真的绷不住
Connections:
- net at U5.~: now also U6.~; no longer U3.~ (~U)
- new net: U1.~ (~U), U2.~ (~U), U3.~ (~U), U4.~ (~U), U5.~
- new net: U1.~ (~U), U2.~ (~U), U3.~ (~U), U4.~ (~U), U6.~
- new net: U1.~ (~U), U5.~, U5.~, U6.~
- new net: U2.~ (~U), U5.~, U6.~
- new net: U3.~ (~U), U5.~
- new net: U4.~ (~U), U5.~
- new net ~CS2: JP1.~ (~CS2)
- no-connect marks 7 -> 6
Other:
- note added: "/CS"
- note added: "/RD"
- note added: "A0-A23\n"
- note added: "D0-D15\n"
- moved on the sheet: C1, JP1, U1, U2, U3, U4, U5A, U5B, U5C, U5D, U6A, U6B
